Commit message: Vision py working

File: intelligent_drone/sensors/sonar_sensor.urdf.xacro (robot description, xacro)
@@ -32,5 +32,5 @@
       <sensor type="ray" name="${name}">
         <update_rate>${update_rate}</update_rate>
-        <visualize>true</visualize>
+        <visualize>false</visualize>
         <ray>
           <range>

File: intelligent_drone/urdf/hector_camera_laser.urdf.xacro (robot description, xacro)
@@ -13,5 +13,5 @@
                           cam_info_topic="front_cam/camera_info" update_rate="10" res_x="1280" res_y="1080"
                           image_format="R8G8B8" hfov="90">
-      <origin xyz="0.4 0 0 " rpy="0 0.57 0"/>
+      <origin xyz="0.4 0 0 " rpy="0 1.57 0"/>
     </xacro:generic_camera>
     <xacro:include filename="$(find hector_quadrotor_gazebo)/urdf/quadrotor_plugins.gazebo.xacro" />
